File: GPS_mk2/GPS_module_mk2/GPS_mk2.sch (EAGLE design)
At the start: 12 parts

Commit message: bunch of stuff I forgot to commit
Parts:
- removed U$10: (no value), 000_CustomPartsMaster:RESISTOR
- removed U$11, U$12, U$13: (no value), 000_CustomPartsMaster:CAPACITOR-UNPOLARIZED0805
- removed U$3: 100nF, 000_CustomPartsMaster:CAPACITOR-UNPOLARIZED0805
- removed U$7, U$8, U$9: 10k, 000_CustomPartsMaster:RESISTOR
- removed U_INS: U_INS, 000_CustomPartsMaster:U_INS
- added C1, C2, C3, C4, C5, C6, C7: (no value), 000_CustomPartsMaster:CAPACITOR-UNPOLARIZED0805
- added GPS_MK2: SENSOR_MODULE_MK1, 000_CustomPartsMaster:SENSOR_MODULE_MK1
- added IC1: MAX3232CSE, maxim:MAX3232CSE
- added R1, U$2, U$5: (no value), 000_CustomPartsMaster:RESISTOR
- U$1: value SENSOR_MODULE_MK1 -> (none); device 000_CustomPartsMaster:SENSOR_MODULE_MK1 -> 000_CustomPartsMaster:RESISTOR
- U$6: value 10k -> (none)
Connections:
- removed net GPS_RX: U$4.PD1_(PCINT17,TXD), U_INS.G6/SV5/MOSI/RX1
- removed net GPS_TX: U$4.PD0_(PCINT16,RXD), U_INS.G7/MISO/TX1
- removed net TIMEPULSE: U_INS.TIMEPULSE
- new net N$1: C1.P$2, IC1G$1.C1+
- new net N$10: GPS_MK2.CMDLED_ANODE, U$6.P$2
- new net N$11: C3.P$2, IC1G$1.V+
- new net N$2: C2.P$1, IC1G$1.C2+
- new net N$6: C4.P$2, IC1G$1.V-
- new net N$9: GPS_MK2.PINGLED_ANODE, U$5.P$2
- new net RCV: GPS_MK2.DATA1/SCL/RX, IC1G$1.R1IN
- new net RCV_TTL: IC1G$1.R1OUT, U$4.PD0_(PCINT16,RXD)
- new net TXD: GPS_MK2.DATA0/SDA/TX, IC1G$1.T1OUT
- new net TXD_TTL: IC1G$1.T1IN, U$4.PD1_(PCINT17,TXD)
- net 3P3V: now also C5.P$1, C6.P$2, C7.P$2, GPS_MK2.3P3PV@1, GPS_MK2.3P3V@3, IC1P.VCC, R1.P$1, U$1.P$1; no longer U$1.3P3PV@1, U$1.3P3V@3, U$10.P$1, U$11.P$2, U$12.P$2, U$13.P$2, U$3.P$1, U$6.P$1, U_INS.GPS.VBAT, U_INS.VCC
- net ALIVE: now also U$2.P$1; no longer U$7.P$1
- net CMD: now also U$6.P$1; no longer U$9.P$1
- net GND: now also C3.P$1, C4.P$1, C5.P$2, C6.P$1, C7.P$1, GPS_MK2.ALIVELED_CATHODE, GPS_MK2.CMDLED_CATHODE, GPS_MK2.GND@1, GPS_MK2.GND@3, GPS_MK2.PINGLED_CATHODE, GPS_MK2.PWRLED_CATHODE, IC1P.GND; no longer U$1.ALIVELED_CATHODE, U$1.CMDLED_CATHODE, U$1.GND@1, U$1.GND@3, U$1.PINGLED_CATHODE, U$1.PWRLED_CATHODE, U$11.P$1, U$12.P$1, U$13.P$1, U$3.P$2, U_INS.GND0, U_INS.GND1
- net MISO: now also GPS_MK2.MISO; no longer U$1.MISO
- net MOSI: now also GPS_MK2.MOSI; no longer U$1.MOSI
- net N$3: now also C1.P$1, IC1G$1.C1-; no longer U$1.PWRLED_ANODE, U$6.P$2
- net N$4: now also C2.P$2, IC1G$1.C2-; no longer U$1.ALIVELED_ANODE, U$7.P$2
- net N$7: now also GPS_MK2.ALIVELED_ANODE, U$2.P$2; no longer U$1.PINGLED_ANODE, U$8.P$2
- net N$8: now also GPS_MK2.PWRLED_ANODE, U$1.P$2; no longer U$1.CMDLED_ANODE, U$9.P$2
- net PING: now also U$5.P$1; no longer U$8.P$1
- net RESET: now also GPS_MK2.!RESET, GPS_MK2.RESET, R1.P$2; no longer U$1.!RESET, U$1.RESET, U$10.P$2
- net SCK: now also GPS_MK2.SCK; no longer U$1.SCK
- net SCL: now also GPS_MK2.SCL; no longer U$1.SCL
- net SDA: now also GPS_MK2.SDA; no longer U$1.SDA
Other:
- moved on the sheet: U$4, U$6

Commit message: IMU layout. GPS layout tweaks
Parts:
- GPS: value SENSOR_MODULE_MK1 -> MK2
- renumbered GPS_MK2 to GPS
Changed lines of the file:
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@@
 <?xml version="1.0" encoding="utf-8"?>
 <!DOCTYPE eagle SYSTEM "eagle.dtd">
-<eagle version="8.3.2">
+<eagle version="8.4.0">
 <drawing>
 <settings>
@@
 <part name="C1" library="000_CustomPartsMaster" deviceset="CAPACITOR-UNPOLARIZED" device="0805"/>
 <part name="C2" library="000_CustomPartsMaster" deviceset="CAPACITOR-UNPOLARIZED" device="0805"/>
-<part name="GPS_MK2" library="000_CustomPartsMaster" deviceset="SENSOR_MODULE_MK1" device=""/>
+<part name="GPS" library="000_CustomPartsMaster" deviceset="SENSOR_MODULE_MK1" device="" value="MK2"/>
 <part name="U$4" library="000_CustomPartsMaster" deviceset="ATMEGA328" device="TQFP32-08"/>
 <part name="U$1" library="000_CustomPartsMaster" deviceset="RESISTOR" device=""/>
@@
 <instance part="C1" gate="G$1" x="-2.54" y="165.1" rot="R90"/>
 <instance part="C2" gate="G$1" x="-2.54" y="154.94" rot="R270"/>
-<instance part="GPS_MK2" gate="G$1" x="81.28" y="48.26"/>
+<instance part="GPS" gate="G$1" x="81.28" y="48.26"/>
 <instance part="U$4" gate="G$1" x="-55.88" y="142.24" rot="R180"/>
 <instance part="U$1" gate="G$1" x="78.74" y="175.26" rot="R90"/>
@@
 <net name="3P3V" class="0">
 <segment>
-<pinref part="GPS_MK2" gate="G$1" pin="3P3PV@1"/>
+<pinref part="GPS" gate="G$1" pin="3P3PV@1"/>
 <wire x1="101.6" y1="111.76" x2="96.52" y2="111.76" width="0.1524" layer="91"/>
 <label x="96.52" y="111.76" size="1.778" layer="95" rot="R180" xref="yes"/>
@@
 </segment>
 <segment>
-<pinref part="GPS_MK2" gate="G$1" pin="3P3V@3"/>
+<pinref part="GPS" gate="G$1" pin="3P3V@3"/>
 <wire x1="101.6" y1="25.4" x2="91.44" y2="25.4" width="0.1524" layer="91"/>
 <label x="91.44" y="25.4" size="1.778" layer="95"/>
@@
 <net name="GND" class="0">
 <segment>
-<pinref part="GPS_MK2" gate="G$1" pin="GND@1"/>
+<pinref part="GPS" gate="G$1" pin="GND@1"/>
 <wire x1="101.6" y1="109.22" x2="96.52" y2="109.22" width="0.1524" layer="91"/>
 <label x="96.52" y="109.22" size="1.778" layer="95" rot="R180" xref="yes"/>
@@
 </segment>
 <segment>
-<pinref part="GPS_MK2" gate="G$1" pin="PWRLED_CATHODE"/>
-<pinref part="GPS_MK2" gate="G$1" pin="ALIVELED_CATHODE"/>
+<pinref part="GPS" gate="G$1" pin="PWRLED_CATHODE"/>
+<pinref part="GPS" gate="G$1" pin="ALIVELED_CATHODE"/>
 <wire x1="101.6" y1="175.26" x2="101.6" y2="160.02" width="0.1524" layer="91"/>
-<pinref part="GPS_MK2" gate="G$1" pin="PINGLED_CATHODE"/>
+<pinref part="GPS" gate="G$1" pin="PINGLED_CATHODE"/>
 <wire x1="101.6" y1="160.02" x2="101.6" y2="144.78" width="0.1524" layer="91"/>
 <junction x="101.6" y="160.02"/>
-<pinref part="GPS_MK2" gate="G$1" pin="CMDLED_CATHODE"/>
+<pinref part="GPS" gate="G$1" pin="CMDLED_CATHODE"/>
 <wire x1="101.6" y1="129.54" x2="101.6" y2="144.78" width="0.1524" layer="91"/>
 <junction x="101.6" y="144.78"/>
@@
 </segment>
 <segment>
-<pinref part="GPS_MK2" gate="G$1" pin="GND@3"/>
+<pinref part="GPS" gate="G$1" pin="GND@3"/>
 <wire x1="101.6" y1="12.7" x2="91.44" y2="12.7" width="0.1524" layer="91"/>
 <label x="91.44" y="12.7" size="1.778" layer="95"/>
@@
 <net name="RESET" class="0">
 <segment>
-<pinref part="GPS_MK2" gate="G$1" pin="!RESET"/>
+<pinref part="GPS" gate="G$1" pin="!RESET"/>
 <wire x1="101.6" y1="96.52" x2="99.06" y2="96.52" width="0.1524" layer="91"/>
 <label x="88.9" y="96.52" size="1.778" layer="95"/>
@@
 </segment>
 <segment>
-<pinref part="GPS_MK2" gate="G$1" pin="RESET"/>
+<pinref part="GPS" gate="G$1" pin="RESET"/>
 <wire x1="101.6" y1="15.24" x2="91.44" y2="15.24" width="0.1524" layer="91"/>
 <label x="91.44" y="15.24" size="1.778" layer="95"/>
@@
 <net name="SCL" class="0">
 <segment>
-<pinref part="GPS_MK2" gate="G$1" pin="SCL"/>
+<pinref part="GPS" gate="G$1" pin="SCL"/>
 <wire x1="101.6" y1="73.66" x2="88.9" y2="73.66" width="0.1524" layer="91"/>
 <label x="88.9" y="73.66" size="1.778" layer="95"/>
@@
 <segment>
 <pinref part="U$2" gate="G$1" pin="P$2"/>
-<pinref part="GPS_MK2" gate="G$1" pin="ALIVELED_ANODE"/>
+<pinref part="GPS" gate="G$1" pin="ALIVELED_ANODE"/>
 <wire x1="83.82" y1="160.02" x2="88.9" y2="160.02" width="0.1524" layer="91"/>
 </segment>
@@
 <segment>
 <pinref part="U$1" gate="G$1" pin="P$2"/>
-<pinref part="GPS_MK2" gate="G$1" pin="PWRLED_ANODE"/>
+<pinref part="GPS" gate="G$1" pin="PWRLED_ANODE"/>
 <wire x1="83.82" y1="175.26" x2="88.9" y2="175.26" width="0.1524" layer="91"/>
 </segment>
@@
 <segment>
 <pinref part="U$5" gate="G$1" pin="P$2"/>
-<pinref part="GPS_MK2" gate="G$1" pin="PINGLED_ANODE"/>
+<pinref part="GPS" gate="G$1" pin="PINGLED_ANODE"/>
 <wire x1="83.82" y1="144.78" x2="88.9" y2="144.78" width="0.1524" layer="91"/>
 </segment>
@@
 <segment>
 <pinref part="U$6" gate="G$1" pin="P$2"/>
-<pinref part="GPS_MK2" gate="G$1" pin="CMDLED_ANODE"/>
+<pinref part="GPS" gate="G$1" pin="CMDLED_ANODE"/>
 <wire x1="83.82" y1="129.54" x2="88.9" y2="129.54" width="0.1524" layer="91"/>
 </segment>
@@
 </segment>
 <segment>
-<pinref part="GPS_MK2" gate="G$1" pin="DATA0/SDA/TX"/>
+<pinref part="GPS" gate="G$1" pin="DATA0/SDA/TX"/>
 <wire x1="101.6" y1="43.18" x2="91.44" y2="43.18" width="0.1524" layer="91"/>
 <label x="91.44" y="43.18" size="1.778" layer="95"/>
@@
 </segment>
 <segment>
-<pinref part="GPS_MK2" gate="G$1" pin="DATA1/SCL/RX"/>
+<pinref part="GPS" gate="G$1" pin="DATA1/SCL/RX"/>
 <wire x1="101.6" y1="40.64" x2="91.44" y2="40.64" width="0.1524" layer="91"/>
 <label x="91.44" y="40.64" size="1.778" layer="95"/>
@@
 </segment>
 <segment>
-<pinref part="GPS_MK2" gate="G$1" pin="MOSI"/>
+<pinref part="GPS" gate="G$1" pin="MOSI"/>
 <wire x1="101.6" y1="20.32" x2="91.44" y2="20.32" width="0.1524" layer="91"/>
 <label x="91.44" y="20.32" size="1.778" layer="95"/>
@@
 </segment>
 <segment>
-<pinref part="GPS_MK2" gate="G$1" pin="MISO"/>
+<pinref part="GPS" gate="G$1" pin="MISO"/>
 <wire x1="101.6" y1="22.86" x2="91.44" y2="22.86" width="0.1524" layer="91"/>
 <label x="91.44" y="22.86" size="1.778" layer="95"/>
@@
 </segment>
 <segment>
-<pinref part="GPS_MK2" gate="G$1" pin="SCK"/>
+<pinref part="GPS" gate="G$1" pin="SCK"/>
 <wire x1="101.6" y1="17.78" x2="91.44" y2="17.78" width="0.1524" layer="91"/>
 <label x="91.44" y="17.78" size="1.778" layer="95"/>
@@
 </segment>
 <segment>
-<pinref part="GPS_MK2" gate="G$1" pin="SDA"/>
+<pinref part="GPS" gate="G$1" pin="SDA"/>
 <wire x1="101.6" y1="76.2" x2="88.9" y2="76.2" width="0.1524" layer="91"/>
 <label x="88.9" y="76.2" size="1.778" layer="95"/>
