File: IMU_mk1/brd/imu_mk1.brd (EAGLE design)
At the start: 38.1 x 38.1 mm, 12 parts

Commit message: bunch of stuff I forgot to commit
Parts:
- removed U$10, U$11, U$12, U$13: (no value), 000_CustomPartsMaster:0805_STACKPOLERESISTOR
- removed U$8, U$9: 10k, 000_CustomPartsMaster:0805_STACKPOLERESISTOR
- removed U_INS: U_INS, 000_CustomPartsMaster:U_INS
- added IMU_MK2: SENSOR_MODULE_MK1, 000_CustomPartsMaster:SENSOR_MODULE_MK1
- added U$5: (no value), 000_CustomPartsMaster:0805_STACKPOLERESISTOR
- added U100: ATMEGA328PB, StevenV1:TQFP32-08
- U$1: value SENSOR_MODULE_MK1 -> 4PIN-HEADER; device 000_CustomPartsMaster:SENSOR_MODULE_MK1 -> 000_CustomPartsMaster:4HEADER_10MIL
- U$3: value 100nF -> (none)
- U$4: value ATMEGA328TQFP32-08 -> (none); device 000_CustomPartsMaster:TQFP32-08 -> 000_CustomPartsMaster:0805_STACKPOLERESISTOR
- U$6, U$7: value 10k -> (none)
- moved U$1 23.6 mm to (19.1, 14.0), turned to 90 degrees
- moved U$3 18.7 mm to (27.9, 29.2), turned to 0 degrees
- moved U$6 10.7 mm to (27.9, 21.6)
- moved U$4 10.6 mm to (27.9, 26.7), turned to 0 degrees
- moved U$7 1.80 mm to (27.9, 31.8), turned to 180 degrees
Connections:
- removed net GPS_RX: U$4.31, U_INS.G6/RX1/MOSI
- removed net GPS_TX: U$4.30, U_INS.G7/TX1/MISO
- removed net N$7: U$1.PINGLED_ANODE, U$8.P$2
- removed net N$8: U$1.CMDLED_ANODE, U$9.P$2
- removed net SCL: U$1.SCL, U$4.28
- removed net SDA: U$1.SDA, U$4.27
- removed net TIMEPULSE: U_INS.GPS.TIMEPULSE
- new net N$1: IMU_MK2.PWRLED_ANODE, U$3.P$2
- new net N$2: IMU_MK2.ALIVELED_ANODE, U$4.P$2
- new net SCL0: IMU_MK2.SCL, U100.28
- new net SCL1: U$1.P$4, U100.6
- new net SDA0: IMU_MK2.SDA, U100.27
- new net SDA1: U$1.P$3, U100.3
- net 3P3V: now also IMU_MK2.3P3V@1, IMU_MK2.3P3V@4, U$1.P$2, U$7.P$1, U100.18, U100.20, U100.4; no longer U$1.3P3V@1, U$1.3P3V@4, U$10.P$1, U$11.P$2, U$12.P$2, U$13.P$2, U$4.18, U$4.20, U$4.4, U$4.6, U$6.P$1, U_INS.GPS.VBAT, U_INS.VCC
- net ALIVE: now also U$4.P$1; no longer U$4.14, U$7.P$1
- net CMD: now also U$6.P$1; no longer U$4.12, U$9.P$1
- net GND: now also IMU_MK2.ALIVELED_CATHODE, IMU_MK2.CMDLED_CATHODE, IMU_MK2.GND@1, IMU_MK2.GND@4, IMU_MK2.PINGLED_CATHODE, IMU_MK2.PWRLED_CATHODE, U$1.P$1, U100.21, U100.5; no longer U$1.ALIVELED_CATHODE, U$1.CMDLED_CATHODE, U$1.GND@1, U$1.GND@4, U$1.PINGLED_CATHODE, U$1.PWRLED_CATHODE, U$11.P$1, U$12.P$1, U$13.P$1, U$3.P$2, U$4.21, U$4.3, U$4.5, U_INS.GND0, U_INS.GND1
- net MISO: now also IMU_MK2.MISO, U100.16; no longer U$1.MISO, U$4.16
- net MOSI: now also IMU_MK2.MOSI, U100.15; no longer U$1.MOSI, U$4.15
- net N$3: now also IMU_MK2.PINGLED_ANODE, U$5.P$2; no longer U$1.PWRLED_ANODE, U$6.P$2
- net N$4: now also IMU_MK2.CMDLED_ANODE, U$6.P$2; no longer U$1.ALIVELED_ANODE, U$7.P$2
- net PING: now also U$5.P$1; no longer U$4.13, U$8.P$1
- net RESET: now also IMU_MK2.RESET@1, IMU_MK2.RESET@2, U$7.P$2; no longer U$1.RESET@1, U$1.RESET@2, U$10.P$2, U$4.29
- net SCK: now also IMU_MK2.SCK; no longer U$1.SCK, U$4.17
Routing:
- net GND: track 124.5 -> 17.0 mm, vias 3 -> 0
- net 3P3V: track 97.6 -> 32.7 mm, vias 2 -> 0
- net RESET: track 48.6 -> 5.08 mm, vias 3 -> 0
- net SCL0: track 0.00 -> 17.0 mm, vias 0 -> 1
- net MISO: track 16.9 -> 0.00 mm
- net SCL: track 16.1 -> 0.00 mm, vias 1 -> 0
- net SDA: track 15.4 -> 0.00 mm, vias 1 -> 0
- net SCK: track 13.4 -> 0.00 mm
- net ALIVE: track 12.1 -> 0.00 mm
- net PING: track 12.0 -> 0.00 mm
- net SDA0: track 0.00 -> 11.6 mm, vias 0 -> 1
- net CMD: track 11.1 -> 0.00 mm
- net MOSI: track 11.1 -> 0.00 mm
- net N$8: track 8.21 -> 0.00 mm
- net N$7: track 8.21 -> 0.00 mm
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
Commit message: IMU layout. GPS layout tweaks
Parts:
- added U$10, U$2, U$8, U$9: (no value), 000_CustomPartsMaster:0805_STACKPOLERESISTOR
- added U1: 9DoF IMU, SparkFun-Sensors:QFN24-3X3
- IMU: value SENSOR_MODULE_MK1 -> MK1
- U$1: value 4PIN-HEADER -> (none); device 000_CustomPartsMaster:4HEADER_10MIL -> 000_CustomPartsMaster:0805_STACKPOLERESISTOR
- moved U$1 5.68 mm to (16.5, 8.89), turned to 0 degrees
- renumbered IMU_MK2 to IMU
Connections:
- new net REGOUT: U$8.P$2, U1.10
- net 3P3V: now also IMU.3P3V@2, IMU.3P3V@3, U$10.P$2, U$2.P$2, U$9.P$2, U1.1, U1.13, U1.22, U1.8
- net GND: now also IMU.GND@2, IMU.GND@3, U$2.P$1, U$8.P$1, U1.18, U1.20, U1.9
- net SCK: now also U100.17
- net SCL1: now also IMU.DATA1@1, IMU.DATA1@2, U$10.P$1, U1.23; no longer U$1.P$4
- net SDA1: now also IMU.DATA0@1, IMU.DATA0@2, U$9.P$1, U1.24; no longer U$1.P$3
Routing:
- net GND: track 17.0 -> 123.9 mm, vias 0 -> 7
- net 3P3V: track 32.7 -> 112.4 mm, vias 0 -> 6
- net SDA1: track 5.62 -> 41.1 mm
- net SCL1: track 5.73 -> 36.7 mm
- net MISO: track 0.00 -> 26.1 mm, vias 0 -> 1
- net RESET: track 5.08 -> 28.9 mm, vias 0 -> 1
- net SCK: track 0.00 -> 22.2 mm, vias 0 -> 1
- net MOSI: track 0.00 -> 21.7 mm, vias 0 -> 1
- net N$4: track 0.00 -> 8.19 mm
- net N$3: track 0.00 -> 8.19 mm
- net N$2: track 0.00 -> 8.19 mm
- net N$1: track 0.00 -> 8.19 mm
- net REGOUT: track 0.00 -> 3.28 mm
