File: IMU_mk1/brd/imu_mk1.sch (EAGLE design)
At the start: 12 parts

Commit message: bunch of stuff I forgot to commit
Parts:
- removed U$10: (no value), 000_CustomPartsMaster:RESISTOR
- removed U$11, U$12, U$13: (no value), 000_CustomPartsMaster:CAPACITOR-UNPOLARIZED0805
- removed U$8, U$9: 10k, 000_CustomPartsMaster:RESISTOR
- removed U_INS: U_INS, 000_CustomPartsMaster:U_INS
- added IMU_MK2: SENSOR_MODULE_MK1, 000_CustomPartsMaster:SENSOR_MODULE_MK1
- added U$5: (no value), 000_CustomPartsMaster:RESISTOR
- added U100: ATMEGA328PB, StevenV1:ATMEGA328PB
- U$1: value SENSOR_MODULE_MK1 -> 4PIN-HEADER; device 000_CustomPartsMaster:SENSOR_MODULE_MK1 -> 000_CustomPartsMaster:4PIN-HEADER
- U$3: value 100nF -> (none); device 000_CustomPartsMaster:CAPACITOR-UNPOLARIZED0805 -> 000_CustomPartsMaster:RESISTOR
- U$4: value ATMEGA328TQFP32-08 -> (none); device 000_CustomPartsMaster:ATMEGA328TQFP32-08 -> 000_CustomPartsMaster:RESISTOR
- U$6, U$7: value 10k -> (none)
Connections:
- removed net GPS_RX: U$4.PD1_(PCINT17,TXD), U_INS.G6/SV5/MOSI/RX1
- removed net GPS_TX: U$4.PD0_(PCINT16,RXD), U_INS.G7/MISO/TX1
- removed net N$7: U$1.PINGLED_ANODE, U$8.P$2
- removed net N$8: U$1.CMDLED_ANODE, U$9.P$2
- removed net SCL: U$1.SCL, U$4.PC5_(ADC5,SCL,PCINT13)
- removed net SDA: U$1.SDA, U$4.PC4_(ADC4,SDA,PCINT12)
- removed net TIMEPULSE: U_INS.TIMEPULSE
- new net N$1: IMU_MK2.PWRLED_ANODE, U$3.P$2
- new net N$2: IMU_MK2.ALIVELED_ANODE, U$4.P$2
- new net SCL0: IMU_MK2.SCL, U100.28(ADC5/PTCY/SCL0)PC5
- new net SCL1: U$1.P$4, U100.6(SCL1/T4/PTXCY)PE1
- new net SDA0: IMU_MK2.SDA, U100.27(ADC4/PTCY/SDA0)PC4
- new net SDA1: U$1.P$3, U100.3(SDA1/ICP4/AC0/PTCXY)PE0
- net 3P3V: now also IMU_MK2.3P3PV@1, IMU_MK2.3P3V@3, U$1.P$2, U$7.P$1, U100.18AVCC, U100.20AREF, U100.4VCC; no longer U$1.3P3PV@1, U$1.3P3V@3, U$10.P$1, U$11.P$2, U$12.P$2, U$13.P$2, U$4.AREF, U$4.AVCC, U$4.VCC@4, U$4.VCC@6, U$6.P$1, U_INS.GPS.VBAT, U_INS.VCC
- net ALIVE: now also U$4.P$1; no longer U$4.PB2_(!SS,OC1B,PCINT2), U$7.P$1
- net CMD: now also U$6.P$1; no longer U$4.PB0_(PCINT0,CLKO,ICP1), U$9.P$1
- net GND: now also IMU_MK2.ALIVELED_CATHODE, IMU_MK2.CMDLED_CATHODE, IMU_MK2.GND@1, IMU_MK2.GND@3, IMU_MK2.PINGLED_CATHODE, IMU_MK2.PWRLED_CATHODE, U$1.P1, U100.21GND2, U100.5GND; no longer U$1.ALIVELED_CATHODE, U$1.CMDLED_CATHODE, U$1.GND@1, U$1.GND@3, U$1.PINGLED_CATHODE, U$1.PWRLED_CATHODE, U$11.P$1, U$12.P$1, U$13.P$1, U$3.P$2, U$4.GND@21, U$4.GND@3, U$4.GND@5, U_INS.GND0, U_INS.GND1
- net MISO: now also IMU_MK2.MISO, U100.16(MISO0/RXD1/PTCXY)PB4; no longer U$1.MISO, U$4.PB4_(MISO,PCINT4)
- net MOSI: now also IMU_MK2.MOSI, U100.15(MOSI0/TXD1/OC2A/PTCXY)PB3; no longer U$1.MOSI, U$4.PB3_(MOSI,OC2A,PCINT3)
- net N$3: now also IMU_MK2.PINGLED_ANODE, U$5.P$2; no longer U$1.PWRLED_ANODE, U$6.P$2
- net N$4: now also IMU_MK2.CMDLED_ANODE, U$6.P$2; no longer U$1.ALIVELED_ANODE, U$7.P$2
- net PING: now also U$5.P$1; no longer U$4.PB1_(OC1A,PCINT1), U$8.P$1
- net RESET: now also IMU_MK2.!RESET, IMU_MK2.RESET, U$7.P$2; no longer U$1.!RESET, U$1.RESET, U$10.P$2, U$4.PC6_(PCINT14,!RESET)
- net SCK: now also IMU_MK2.SCK; no longer U$1.SCK, U$4.PB5_(SCK,PCINT5)
Other:
- moved on the sheet: U$6, U$7

Commit message: IMU layout. GPS layout tweaks
Parts:
- added U$10, U$9: (no value), 000_CustomPartsMaster:RESISTOR
- added U$2, U$8: (no value), 000_CustomPartsMaster:CAPACITOR-UNPOLARIZED0805
- added U1: 9DoF IMU, SparkFun-Sensors:MPU-9250
- IMU: value SENSOR_MODULE_MK1 -> MK1
- U$1: value 4PIN-HEADER -> (none); device 000_CustomPartsMaster:4PIN-HEADER -> 000_CustomPartsMaster:CAPACITOR-UNPOLARIZED0805
- renumbered IMU_MK2 to IMU
Connections:
- new net REGOUT: U$8.P$2, U1.REGOUT
- net 3P3V: now also IMU.3P3V@2, U$10.P$2, U$2.P$2, U$9.P$2, U1.!CS, U1.VDD, U1.VDDIO
- net GND: now also IMU.GND@2, U$1.P$1, U$2.P$1, U$8.P$1, U1.AD0/SDO, U1.GND; no longer U$1.P1
- net SCK: now also U100.17(PTCXY/XCK0/SCK0)PB5
- net SCL1: now also IMU.DATA1/SCL/RX, U$10.P$1, U1.SCL/SCLK; no longer U$1.P$4
- net SDA1: now also IMU.DATA0/SDA/TX, U$9.P$1, U1.SDA/SDI; no longer U$1.P$3
