File: SHT_mk2/brd/SHT_mk2/SHT Test Module.brd (EAGLE design)
At the start: 38.1 x 38.1 mm, 11 parts, among them U100 ATMEGA328TQFP32-08

Commit message: IMU layout. GPS layout tweaks
Parts:
- SHT: value SENSOR_MODULE_MK1 -> MK2
- renumbered SHT_MK2 to SHT
Routing:
- net 3P3V: track 81.2 -> 75.3 mm
