File: SHT_mk2/brd/SHT_mk2/SHT Test Module.sch (EAGLE design)
At the start: 13 parts

Commit message: bunch of stuff I forgot to commit
Parts:
- removed U$1: SENSOR_MODULE_MK1, 000_CustomPartsMaster:SENSOR_MODULE_MK1
- removed U$10: (no value), 000_CustomPartsMaster:RESISTOR
- removed U$11, U$12, U$13: (no value), 000_CustomPartsMaster:CAPACITOR-UNPOLARIZED0805
- removed U$3: 100nF, 000_CustomPartsMaster:CAPACITOR-UNPOLARIZED0805
- removed U$4: ATMEGA328TQFP32-08, 000_CustomPartsMaster:ATMEGA328TQFP32-08
- removed U$5: (no value), 000_CustomPartsMaster:6PIN-HEADER2X3
- removed U$6, U$7, U$8, U$9: 10k, 000_CustomPartsMaster:RESISTOR
- removed U_INS: U_INS, 000_CustomPartsMaster:U_INS
- added C200, C201, C202: 0.1uF, 000_CustomPartsMaster:CAPACITOR-UNPOLARIZED0805
- added R100, R101, R102, R103: 1k, 000_CustomPartsMaster:RESISTOR
- added R200, R201: 10k, 000_CustomPartsMaster:RESISTOR
- added SHT_MK2: SENSOR_MODULE_MK1, 000_CustomPartsMaster:SENSOR_MODULE_MK1
- added U100: ATMEGA328TQFP32-08, 000_CustomPartsMaster:ATMEGA328TQFP32-08
Connections:
- removed net GPS_RX: U$4.PD1_(PCINT17,TXD), U_INS.G6/SV5/MOSI/RX1
- removed net GPS_TX: U$4.PD0_(PCINT16,RXD), U_INS.G7/MISO/TX1
- removed net N$3: U$1.PWRLED_ANODE, U$6.P$2
- removed net N$4: U$1.ALIVELED_ANODE, U$7.P$2
- removed net N$7: U$1.PINGLED_ANODE, U$8.P$2
- removed net N$8: U$1.CMDLED_ANODE, U$9.P$2
- removed net PWR: U$1.3.3V, U$10.P$1, U$11.P$2, U$12.P$2, U$13.P$2, U$3.P$1, U$4.AREF, U$4.AVCC, U$4.VCC@4, U$4.VCC@6, U$5.P1, U$6.P$1, U_INS.GPS.VBAT, U_INS.VCC
- removed net TIMEPULSE: U_INS.TIMEPULSE
- new net 3P3V: C200.P$2, C201.P$2, C202.P$2, R100.P$1, R200.P$2, R201.P$2, SHT_MK2.3P3PV@1, SHT_MK2.3P3V@2, SHT_MK2.3P3V@3, U100.AREF, U100.AVCC, U100.VCC@4, U100.VCC@6
- new net CLK: SHT_MK2.DATA1/SCL/RX, U100.PC1_(ADC1,PCINT9)
- new net DATA: R201.P$1, SHT_MK2.DATA0/SDA/TX, U100.PC0_(ADC0,PCINT8)
- new net N$12: R100.P$2, SHT_MK2.PWRLED_ANODE
- new net N$13: R101.P$2, SHT_MK2.ALIVELED_ANODE
- new net N$14: R102.P$2, SHT_MK2.PINGLED_ANODE
- new net N$15: R103.P$2, SHT_MK2.CMDLED_ANODE
- net ALIVE: now also R101.P$1, U100.PD0_(PCINT16,RXD); no longer U$4.PB2_(!SS,OC1B,PCINT2), U$7.P$1
- net CMD: now also R103.P$1, U100.PD2_(PCINT18,INT0); no longer U$4.PB0_(PCINT0,CLKO,ICP1), U$9.P$1
- net GND: now also C200.P$1, C201.P$1, C202.P$1, SHT_MK2.ALIVELED_CATHODE, SHT_MK2.CMDLED_CATHODE, SHT_MK2.GND@1, SHT_MK2.GND@2, SHT_MK2.GND@3, SHT_MK2.PINGLED_CATHODE, SHT_MK2.PWRLED_CATHODE, U100.GND@21, U100.GND@3, U100.GND@5; no longer U$1.ALIVELED_CATHODE, U$1.CMDLED_CATHODE, U$1.GND, U$1.PINGLED_CATHODE, U$1.PWRLED_CATHODE, U$11.P$1, U$12.P$1, U$13.P$1, U$3.P$2, U$4.GND@21, U$4.GND@3, U$4.GND@5, U$5.P2, U_INS.GND0, U_INS.GND1
- net MISO: now also SHT_MK2.MISO, U100.PB4_(MISO,PCINT4); no longer U$4.PB4_(MISO,PCINT4), U$5.P4
- net MOSI: now also SHT_MK2.MOSI, U100.PB3_(MOSI,OC2A,PCINT3); no longer U$4.PB3_(MOSI,OC2A,PCINT3), U$5.P3
- net PING: now also R102.P$1, U100.PD1_(PCINT17,TXD); no longer U$4.PB1_(OC1A,PCINT1), U$8.P$1
- net RESET: now also R200.P$1, SHT_MK2.!RESET, SHT_MK2.RESET, U100.PC6_(PCINT14,!RESET); no longer U$1.!RESET, U$10.P$2, U$4.PC6_(PCINT14,!RESET), U$5.P6
- net SCK: now also SHT_MK2.SCK, U100.PB5_(SCK,PCINT5); no longer U$4.PB5_(SCK,PCINT5), U$5.P5
- net SCL: now also SHT_MK2.SCL, U100.PC5_(ADC5,SCL,PCINT13); no longer U$1.SCL, U$4.PC5_(ADC5,SCL,PCINT13)
- net SDA: now also SHT_MK2.SDA, U100.PC4_(ADC4,SDA,PCINT12); no longer U$1.SDA, U$4.PC4_(ADC4,SDA,PCINT12)

Commit message: IMU layout. GPS layout tweaks
Parts:
- SHT: value SENSOR_MODULE_MK1 -> MK2
- renumbered SHT_MK2 to SHT
Changed lines of the file:
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@@
 <?xml version="1.0" encoding="utf-8"?>
 <!DOCTYPE eagle SYSTEM "eagle.dtd">
-<eagle version="8.3.2">
+<eagle version="8.4.0">
 <drawing>
 <settings>
@@
 </classes>
 <parts>
-<part name="SHT_MK2" library="000_CustomPartsMaster" deviceset="SENSOR_MODULE_MK1" device=""/>
+<part name="SHT" library="000_CustomPartsMaster" deviceset="SENSOR_MODULE_MK1" device="" value="MK2"/>
 <part name="U100" library="000_CustomPartsMaster" deviceset="ATMEGA328" device="TQFP32-08"/>
 <part name="R101" library="000_CustomPartsMaster" deviceset="RESISTOR" device="" value="1k"/>
@@
 </plain>
 <instances>
-<instance part="SHT_MK2" gate="G$1" x="99.06" y="0"/>
+<instance part="SHT" gate="G$1" x="99.06" y="0"/>
 <instance part="U100" gate="G$1" x="27.94" y="68.58" rot="R180"/>
 <instance part="R101" gate="G$1" x="99.06" y="111.76" rot="R90"/>
@@
 </segment>
 <segment>
-<pinref part="SHT_MK2" gate="G$1" pin="GND@1"/>
+<pinref part="SHT" gate="G$1" pin="GND@1"/>
 <wire x1="119.38" y1="60.96" x2="111.76" y2="60.96" width="0.1524" layer="91"/>
 <label x="111.76" y="60.96" size="1.778" layer="95" rot="R180" xref="yes"/>
 </segment>
 <segment>
-<pinref part="SHT_MK2" gate="G$1" pin="CMDLED_CATHODE"/>
+<pinref part="SHT" gate="G$1" pin="CMDLED_CATHODE"/>
 <wire x1="119.38" y1="81.28" x2="121.92" y2="81.28" width="0.1524" layer="91"/>
 <label x="121.92" y="81.28" size="1.778" layer="95" xref="yes"/>
 </segment>
 <segment>
-<pinref part="SHT_MK2" gate="G$1" pin="PINGLED_CATHODE"/>
+<pinref part="SHT" gate="G$1" pin="PINGLED_CATHODE"/>
 <wire x1="119.38" y1="96.52" x2="121.92" y2="96.52" width="0.1524" layer="91"/>
 <label x="121.92" y="96.52" size="1.778" layer="95" xref="yes"/>
 </segment>
 <segment>
-<pinref part="SHT_MK2" gate="G$1" pin="ALIVELED_CATHODE"/>
+<pinref part="SHT" gate="G$1" pin="ALIVELED_CATHODE"/>
 <wire x1="119.38" y1="111.76" x2="121.92" y2="111.76" width="0.1524" layer="91"/>
 <label x="121.92" y="111.76" size="1.778" layer="95" xref="yes"/>
@@
 </segment>
 <segment>
-<pinref part="SHT_MK2" gate="G$1" pin="PWRLED_CATHODE"/>
+<pinref part="SHT" gate="G$1" pin="PWRLED_CATHODE"/>
 <wire x1="119.38" y1="127" x2="121.92" y2="127" width="0.1524" layer="91"/>
 <label x="121.92" y="127" size="1.778" layer="95" xref="yes"/>
 </segment>
 <segment>
-<pinref part="SHT_MK2" gate="G$1" pin="GND@2"/>
+<pinref part="SHT" gate="G$1" pin="GND@2"/>
 <wire x1="119.38" y1="-10.16" x2="109.22" y2="-10.16" width="0.1524" layer="91"/>
 <label x="109.22" y="-10.16" size="1.778" layer="95"/>
 </segment>
 <segment>
-<pinref part="SHT_MK2" gate="G$1" pin="GND@3"/>
+<pinref part="SHT" gate="G$1" pin="GND@3"/>
 <wire x1="119.38" y1="-35.56" x2="109.22" y2="-35.56" width="0.1524" layer="91"/>
 <label x="109.22" y="-35.56" size="1.778" layer="95"/>
@@
 <net name="N$12" class="0">
 <segment>
-<pinref part="SHT_MK2" gate="G$1" pin="PWRLED_ANODE"/>
+<pinref part="SHT" gate="G$1" pin="PWRLED_ANODE"/>
 <wire x1="106.68" y1="127" x2="104.14" y2="127" width="0.1524" layer="91"/>
 <pinref part="R100" gate="G$1" pin="P$2"/>
@@
 <net name="N$13" class="0">
 <segment>
-<pinref part="SHT_MK2" gate="G$1" pin="ALIVELED_ANODE"/>
+<pinref part="SHT" gate="G$1" pin="ALIVELED_ANODE"/>
 <wire x1="106.68" y1="111.76" x2="104.14" y2="111.76" width="0.1524" layer="91"/>
 <pinref part="R101" gate="G$1" pin="P$2"/>
@@
 <net name="N$14" class="0">
 <segment>
-<pinref part="SHT_MK2" gate="G$1" pin="PINGLED_ANODE"/>
+<pinref part="SHT" gate="G$1" pin="PINGLED_ANODE"/>
 <wire x1="106.68" y1="96.52" x2="104.14" y2="96.52" width="0.1524" layer="91"/>
 <pinref part="R102" gate="G$1" pin="P$2"/>
@@
 <net name="N$15" class="0">
 <segment>
-<pinref part="SHT_MK2" gate="G$1" pin="CMDLED_ANODE"/>
+<pinref part="SHT" gate="G$1" pin="CMDLED_ANODE"/>
 <wire x1="106.68" y1="81.28" x2="104.14" y2="81.28" width="0.1524" layer="91"/>
 <pinref part="R103" gate="G$1" pin="P$2"/>
@@
 </segment>
 <segment>
-<pinref part="SHT_MK2" gate="G$1" pin="SDA"/>
+<pinref part="SHT" gate="G$1" pin="SDA"/>
 <wire x1="119.38" y1="27.94" x2="111.76" y2="27.94" width="0.1524" layer="91"/>
 <label x="111.76" y="27.94" size="1.778" layer="95" rot="R180" xref="yes"/>
@@
 </segment>
 <segment>
-<pinref part="SHT_MK2" gate="G$1" pin="SCL"/>
+<pinref part="SHT" gate="G$1" pin="SCL"/>
 <wire x1="119.38" y1="25.4" x2="111.76" y2="25.4" width="0.1524" layer="91"/>
 <label x="111.76" y="25.4" size="1.778" layer="95" rot="R180" xref="yes"/>
@@
 </segment>
 <segment>
-<pinref part="SHT_MK2" gate="G$1" pin="!RESET"/>
+<pinref part="SHT" gate="G$1" pin="!RESET"/>
 <wire x1="119.38" y1="48.26" x2="111.76" y2="48.26" width="0.1524" layer="91"/>
 <label x="111.76" y="48.26" size="1.778" layer="95" rot="R180" xref="yes"/>
@@
 </segment>
 <segment>
-<pinref part="SHT_MK2" gate="G$1" pin="RESET"/>
+<pinref part="SHT" gate="G$1" pin="RESET"/>
 <wire x1="119.38" y1="-33.02" x2="109.22" y2="-33.02" width="0.1524" layer="91"/>
 <label x="109.22" y="-33.02" size="1.778" layer="95"/>
@@
 </segment>
 <segment>
-<pinref part="SHT_MK2" gate="G$1" pin="MOSI"/>
+<pinref part="SHT" gate="G$1" pin="MOSI"/>
 <wire x1="119.38" y1="-27.94" x2="109.22" y2="-27.94" width="0.1524" layer="91"/>
 <label x="109.22" y="-27.94" size="1.778" layer="95"/>
@@
 </segment>
 <segment>
-<pinref part="SHT_MK2" gate="G$1" pin="MISO"/>
+<pinref part="SHT" gate="G$1" pin="MISO"/>
 <wire x1="119.38" y1="-25.4" x2="109.22" y2="-25.4" width="0.1524" layer="91"/>
 <label x="109.22" y="-25.4" size="1.778" layer="95"/>
@@
 </segment>
 <segment>
-<pinref part="SHT_MK2" gate="G$1" pin="SCK"/>
+<pinref part="SHT" gate="G$1" pin="SCK"/>
 <wire x1="119.38" y1="-30.48" x2="109.22" y2="-30.48" width="0.1524" layer="91"/>
 <label x="109.22" y="-30.48" size="1.778" layer="95"/>
@@
 </segment>
 <segment>
-<pinref part="SHT_MK2" gate="G$1" pin="DATA0/SDA/TX"/>
+<pinref part="SHT" gate="G$1" pin="DATA0/SDA/TX"/>
 <wire x1="119.38" y1="-5.08" x2="109.22" y2="-5.08" width="0.1524" layer="91"/>
 <label x="109.22" y="-5.08" size="1.778" layer="95"/>
@@
 </segment>
 <segment>
-<pinref part="SHT_MK2" gate="G$1" pin="DATA1/SCL/RX"/>
+<pinref part="SHT" gate="G$1" pin="DATA1/SCL/RX"/>
 <wire x1="119.38" y1="-7.62" x2="109.22" y2="-7.62" width="0.1524" layer="91"/>
 <label x="109.22" y="-7.62" size="1.778" layer="95"/>
@@
 <net name="3P3V" class="0">
 <segment>
-<pinref part="SHT_MK2" gate="G$1" pin="3P3V@2"/>
+<pinref part="SHT" gate="G$1" pin="3P3V@2"/>
 <wire x1="119.38" y1="-2.54" x2="109.22" y2="-2.54" width="0.1524" layer="91"/>
 <label x="109.22" y="-2.54" size="1.778" layer="95"/>
 </segment>
 <segment>
-<pinref part="SHT_MK2" gate="G$1" pin="3P3PV@1"/>
+<pinref part="SHT" gate="G$1" pin="3P3PV@1"/>
 <wire x1="119.38" y1="63.5" x2="111.76" y2="63.5" width="0.1524" layer="91"/>
 <label x="111.76" y="63.5" size="1.778" layer="95" rot="R180" xref="yes"/>
@@
 </segment>
 <segment>
-<pinref part="SHT_MK2" gate="G$1" pin="3P3V@3"/>
+<pinref part="SHT" gate="G$1" pin="3P3V@3"/>
 <wire x1="119.38" y1="-22.86" x2="109.22" y2="-22.86" width="0.1524" layer="91"/>
 <label x="109.22" y="-22.86" size="1.778" layer="95"/>
